File: schematic/connectors.kicad_sch (KiCad schematic)
At the start: 12 parts, among them J2 TSW-104-08-G-T-RA, J3 TSW-104-08-G-T-RA, J4 TSW-104-08-G-T-RA, J5 Conn_01x03, J6 Conn_01x03, J7 USB_B_Micro, Q1 2N7002P_215

Commit message: Complete schematic
Parts:
- removed Q1: 2N7002P_215, Package_TO_SOT_SMD:SOT-23, symbol dk_Transistors-FETs-MOSFETs-Single:2N7002P_215
- added J8: Conn_01x03, JST_New:JST_ZH_B3B-ZR_1x03_P1.50mm_Vertical, symbol Connector_Generic:Conn_01x03
- added Q1: 2N7002P_215, digikey:SOT-23-3, symbol Digikey:2N7002P_215
- R6, R7, R8, R9: footprint (none) -> Resistor_SMD:R_0603_1608Metric
Connections:
- net +3V3: now also J8.1 (Pin_1)
- net GND: now also Q1.2 (S)
- net at R7.2: now also Q1.1 (G)
- net at J5.2 (Pin_2), J6.2 (Pin_2): now also J8.2 (Pin_2), Q1.3 (D)
- net CH10 renamed CH10_SBUS3
- net CH9 renamed CH9_SBUS4
- new net SAT3_RX: J8.3 (Pin_3)
Other:
- moved on the sheet: J6

Commit message: Initial pcb layout - footprints only
Connections:
- net CH1: now also J4.10; no longer J4.1
- net CH10_SBUS3: now also J2.7; no longer J2.4
- net CH11_SBUS2: now also J2.4; no longer J2.7
- net CH12_SBUS1: now also J2.1; no longer J2.10
- net CH2: now also J4.7; no longer J4.4
- net CH3: now also J4.4; no longer J4.7
- net CH4: now also J4.1; no longer J4.10
- net CH5: now also J3.10; no longer J3.1
- net CH6: now also J3.7; no longer J3.4
- net CH7: now also J3.4; no longer J3.7
- net CH8: now also J3.1; no longer J3.10
- net CH9_SBUS4: now also J2.10; no longer J2.1
